Commit message: mark4

File: drob_control/urdf/drob/action/wheel.urdf.xacro (robot description, xacro)
@@ -6,12 +6,12 @@
     <inertial>
       <origin xyz="0 0 0" rpy="0 0 0" />
-      <mass value="0.8" />
-      <inertia
-        ixx="0.001"
-        ixy="0"
-        ixz="0"
-        iyy="0.001"
-        iyz="0"
-        izz="0.001" />
+      <mass value="2.0" />
+      <inertia
+        ixx="0.01"
+        ixy="0"
+        ixz="0"
+        iyy="0.01"
+        iyz="0"
+        izz="0.01" />
     </inertial>
     <visual>
@@ -32,12 +32,12 @@
     <inertial>
       <origin xyz="0 0 0" rpy="0 0 0" />
-      <mass value="0.8" />
-      <inertia
-        ixx="0.001"
-        ixy="0"
-        ixz="0"
-        iyy="0.001"
-        iyz="0"
-        izz="0.001" />
+      <mass value="2.0" />
+      <inertia
+        ixx="0.01"
+        ixy="0"
+        ixz="0"
+        iyy="0.01"
+        iyz="0"
+        izz="0.01" />
     </inertial>
     <visual>
@@ -58,12 +58,12 @@
     <inertial>
       <origin xyz="0 0 0" rpy="0 0 0" />
-      <mass value="0.8" />
-      <inertia
-        ixx="0.001"
-        ixy="0"
-        ixz="0"
-        iyy="0.001"
-        iyz="0"
-        izz="0.001" />
+      <mass value="2.0" />
+      <inertia
+        ixx="0.01"
+        ixy="0"
+        ixz="0"
+        iyy="0.01"
+        iyz="0"
+        izz="0.01" />
     </inertial>
     <visual>
@@ -84,12 +84,12 @@
     <inertial>
       <origin xyz="0 0 0" rpy="0 0 0" />
-      <mass value="0.8" />
-      <inertia
-        ixx="0.001"
-        ixy="0"
-        ixz="0"
-        iyy="0.001"
-        iyz="0"
-        izz="0.001" />
+      <mass value="2.0" />
+      <inertia
+        ixx="0.01"
+        ixy="0"
+        ixz="0"
+        iyy="0.01"
+        iyz="0"
+        izz="0.01" />
     </inertial>
     <visual>
@@ -113,4 +113,5 @@
     <child link="rfw" />
     <axis xyz="0 0 -1" />
+    <dynamics damping="0.1" friction="0.1" />
   </joint>
   <joint name="lfj" type="continuous">
@@ -119,4 +120,5 @@
     <child link="lfw" />
     <axis xyz="0 0 -1" />
+    <dynamics damping="0.1" friction="0.1" />
   </joint>
   <joint name="rbj" type="continuous">
@@ -125,4 +127,5 @@
     <child link="rbw" />
     <axis xyz="0 0 -1" />
+    <dynamics damping="0.1" friction="0.1" />
   </joint>
   <joint name="lbj" type="continuous">
@@ -131,41 +134,99 @@
     <child link="lbw" />
     <axis xyz="0 0 -1" />
+    <dynamics damping="0.1" friction="0.1" />
   </joint>
   <!-- Gazebo标签 -->
   <gazebo reference="rfw">
     <material>Gazebo/Black</material>
-    <mu1>0.8</mu1>
-    <mu2>0.8</mu2>
-    <kp>1000000.0</kp>
-    <kd>50.0</kd>
-    <selfCollide>false</selfCollide>
-    <minDepth>0.001</minDepth>
+    <mu1>1.0</mu1>
+    <mu2>1.0</mu2>
+    <kp>1000000.0</kp>
+    <kd>10.0</kd>
+    <selfCollide>false</selfCollide>
+    <minDepth>0.001</minDepth>
+    <maxVel>20.0</maxVel>
+    <inertia>
+      <ixx>0.01</ixx>
+      <ixy>0</ixy>
+      <ixz>0</ixz>
+      <iyy>0.01</iyy>
+      <iyz>0</iyz>
+      <izz>0.01</izz>
+    </inertia>
+    <gravity>true</gravity>
   </gazebo>
   <gazebo reference="lfw">
     <material>Gazebo/Black</material>
-    <mu1>0.8</mu1>
-    <mu2>0.8</mu2>
-    <kp>1000000.0</kp>
-    <kd>50.0</kd>
-    <selfCollide>false</selfCollide>
-    <minDepth>0.001</minDepth>
+    <mu1>1.0</mu1>
+    <mu2>1.0</mu2>
+    <kp>1000000.0</kp>
+    <kd>10.0</kd>
+    <selfCollide>false</selfCollide>
+    <minDepth>0.001</minDepth>
+    <maxVel>20.0</maxVel>
+    <inertia>
+      <ixx>0.01</ixx>
+      <ixy>0</ixy>
+      <ixz>0</ixz>
+      <iyy>0.01</iyy>
+      <iyz>0</iyz>
+      <izz>0.01</izz>
+    </inertia>
+    <gravity>true</gravity>
   </gazebo>
   <gazebo reference="rbw">
     <material>Gazebo/Black</material>
-    <mu1>0.8</mu1>
-    <mu2>0.8</mu2>
-    <kp>1000000.0</kp>
-    <kd>50.0</kd>
-    <selfCollide>false</selfCollide>
-    <minDepth>0.001</minDepth>
+    <mu1>1.0</mu1>
+    <mu2>1.0</mu2>
+    <kp>1000000.0</kp>
+    <kd>10.0</kd>
+    <selfCollide>false</selfCollide>
+    <minDepth>0.001</minDepth>
+    <maxVel>20.0</maxVel>
+    <inertia>
+      <ixx>0.01</ixx>
+      <ixy>0</ixy>
+      <ixz>0</ixz>
+      <iyy>0.01</iyy>
+      <iyz>0</iyz>
+      <izz>0.01</izz>
+    </inertia>
+    <gravity>true</gravity>
   </gazebo>
   <gazebo reference="lbw">
     <material>Gazebo/Black</material>
-    <mu1>0.8</mu1>
-    <mu2>0.8</mu2>
-    <kp>1000000.0</kp>
-    <kd>50.0</kd>
-    <selfCollide>false</selfCollide>
-    <minDepth>0.001</minDepth>
+    <mu1>1.0</mu1>
+    <mu2>1.0</mu2>
+    <kp>1000000.0</kp>
+    <kd>10.0</kd>
+    <selfCollide>false</selfCollide>
+    <minDepth>0.001</minDepth>
+    <maxVel>20.0</maxVel>
+    <inertia>
+      <ixx>0.01</ixx>
+      <ixy>0</ixy>
+      <ixz>0</ixz>
+      <iyy>0.01</iyy>
+      <iyz>0</iyz>
+      <izz>0.01</izz>
+    </inertia>
+    <gravity>true</gravity>
+  </gazebo>
+  <!-- 为轮子关节添加Gazebo插件 -->
+  <gazebo reference="rfj">
+    <provideFeedback>true</provideFeedback>
+    <implicitSpringDamper>0</implicitSpringDamper>
+  </gazebo>
+  <gazebo reference="lfj">
+    <provideFeedback>true</provideFeedback>
+    <implicitSpringDamper>0</implicitSpringDamper>
+  </gazebo>
+  <gazebo reference="rbj">
+    <provideFeedback>true</provideFeedback>
+    <implicitSpringDamper>0</implicitSpringDamper>
+  </gazebo>
+  <gazebo reference="lbj">
+    <provideFeedback>true</provideFeedback>
+    <implicitSpringDamper>0</implicitSpringDamper>
   </gazebo>
 </robot>

File: drob_control/urdf/drob/drob.control.xacro (robot description, xacro)
@@ -67,9 +67,24 @@
                 <parameters>$(find drob_control)/config/controllers.yaml</parameters>
                 <ros>
-                    <remapping>/drob_diff_drive_controller/cmd_vel_unstamped:=/cmd_vel</remapping>
-                    <remapping>/drob_diff_drive_controller/odom:=/odom</remapping>
+                    <remapping>/drob_left_front_velocity_controller/commands:=/drob_left_front_velocity_controller/commands</remapping>
+                    <remapping>/drob_right_front_velocity_controller/commands:=/drob_right_front_velocity_controller/commands</remapping>
+                    <remapping>/drob_left_back_velocity_controller/commands:=/drob_left_back_velocity_controller/commands</remapping>
+                    <remapping>/drob_right_back_velocity_controller/commands:=/drob_right_back_velocity_controller/commands</remapping>
                 </ros>
             </plugin>
         </gazebo>
+        <!-- 为每个轮子关节添加Gazebo插件 -->
+        <gazebo reference="lfj">
+            <provideFeedback>true</provideFeedback>
+        </gazebo>
+        <gazebo reference="lbj">
+            <provideFeedback>true</provideFeedback>
+        </gazebo>
+        <gazebo reference="rfj">
+            <provideFeedback>true</provideFeedback>
+        </gazebo>
+        <gazebo reference="rbj">
+            <provideFeedback>true</provideFeedback>
+        </gazebo>
     </xacro:macro>
 </robot>

Commit message: mark9(仿真成功前轮无驱动力)

File: drob_control/urdf/drob/action/wheel.urdf.xacro (robot description, xacro)
@@ -2,5 +2,5 @@
 <!-- 汽车轮子 xacro 文件 -->
 <robot xmlns:xacro="http://www.ros.org/wiki/xacro">
-  <!-- 四个轮子链接 -->
+  <!-- 恢复前轮，但配置为无阻力的从动轮 -->
   <link name="rfw">
     <inertial>
@@ -107,5 +107,5 @@
     </collision>
   </link>
-  <!-- 四个轮子关节 -->
+  <!-- 前轮关节 - 配置为极低摩擦的自由转动 -->
   <joint name="rfj" type="continuous">
     <origin xyz="-0.2 -0.15 -0.09" rpy="1.5708 0 0" />
@@ -113,5 +113,5 @@
     <child link="rfw" />
     <axis xyz="0 0 -1" />
-    <dynamics damping="0.1" friction="0.1" />
+    <dynamics damping="0.001" friction="0.001" />
   </joint>
   <joint name="lfj" type="continuous">
@@ -120,5 +120,5 @@
     <child link="lfw" />
     <axis xyz="0 0 -1" />
-    <dynamics damping="0.1" friction="0.1" />
+    <dynamics damping="0.001" friction="0.001" />
   </joint>
   <joint name="rbj" type="continuous">
@@ -127,5 +127,5 @@
     <child link="rbw" />
     <axis xyz="0 0 -1" />
-    <dynamics damping="0.1" friction="0.1" />
+    <dynamics damping="0.2" friction="0.15" />
   </joint>
   <joint name="lbj" type="continuous">
@@ -134,8 +134,47 @@
     <child link="lbw" />
     <axis xyz="0 0 -1" />
-    <dynamics damping="0.1" friction="0.1" />
+    <dynamics damping="0.2" friction="0.15" />
   </joint>
   <!-- Gazebo标签 -->
+  <!-- 前轮Gazebo配置 - 极低摩擦力 -->
   <gazebo reference="rfw">
+    <material>Gazebo/Black</material>
+    <mu1>0.001</mu1>
+    <mu2>0.001</mu2>
+    <kp>1000000.0</kp>
+    <kd>10.0</kd>
+    <selfCollide>false</selfCollide>
+    <minDepth>0.001</minDepth>
+    <maxVel>20.0</maxVel>
+    <inertia>
+      <ixx>0.01</ixx>
+      <ixy>0</ixy>
+      <ixz>0</ixz>
+      <iyy>0.01</iyy>
+      <iyz>0</iyz>
+      <izz>0.01</izz>
+    </inertia>
+    <gravity>true</gravity>
+  </gazebo>
+  <gazebo reference="lfw">
+    <material>Gazebo/Black</material>
+    <mu1>0.001</mu1>
+    <mu2>0.001</mu2>
+    <kp>1000000.0</kp>
+    <kd>10.0</kd>
+    <selfCollide>false</selfCollide>
+    <minDepth>0.001</minDepth>
+    <maxVel>20.0</maxVel>
+    <inertia>
+      <ixx>0.01</ixx>
+      <ixy>0</ixy>
+      <ixz>0</ixz>
+      <iyy>0.01</iyy>
+      <iyz>0</iyz>
+      <izz>0.01</izz>
+    </inertia>
+    <gravity>true</gravity>
+  </gazebo>
+  <gazebo reference="rbw">
     <material>Gazebo/Black</material>
     <mu1>1.0</mu1>
@@ -156,5 +195,5 @@
     <gravity>true</gravity>
   </gazebo>
-  <gazebo reference="lfw">
+  <gazebo reference="lbw">
     <material>Gazebo/Black</material>
     <mu1>1.0</mu1>
@@ -175,43 +214,5 @@
     <gravity>true</gravity>
   </gazebo>
-  <gazebo reference="rbw">
-    <material>Gazebo/Black</material>
-    <mu1>1.0</mu1>
-    <mu2>1.0</mu2>
-    <kp>1000000.0</kp>
-    <kd>10.0</kd>
-    <selfCollide>false</selfCollide>
-    <minDepth>0.001</minDepth>
-    <maxVel>20.0</maxVel>
-    <inertia>
-      <ixx>0.01</ixx>
-      <ixy>0</ixy>
-      <ixz>0</ixz>
-      <iyy>0.01</iyy>
-      <iyz>0</iyz>
-      <izz>0.01</izz>
-    </inertia>
-    <gravity>true</gravity>
-  </gazebo>
-  <gazebo reference="lbw">
-    <material>Gazebo/Black</material>
-    <mu1>1.0</mu1>
-    <mu2>1.0</mu2>
-    <kp>1000000.0</kp>
-    <kd>10.0</kd>
-    <selfCollide>false</selfCollide>
-    <minDepth>0.001</minDepth>
-    <maxVel>20.0</maxVel>
-    <inertia>
-      <ixx>0.01</ixx>
-      <ixy>0</ixy>
-      <ixz>0</ixz>
-      <iyy>0.01</iyy>
-      <iyz>0</iyz>
-      <izz>0.01</izz>
-    </inertia>
-    <gravity>true</gravity>
-  </gazebo>
-  <!-- 为轮子关节添加Gazebo插件 -->
+  <!-- 前轮关节的Gazebo插件 - 自由转动 -->
   <gazebo reference="rfj">
     <provideFeedback>true</provideFeedback>

File: drob_control/urdf/drob/drob.control.xacro (robot description, xacro)
@@ -6,5 +6,5 @@
                 <plugin>gazebo_ros2_control/GazeboSystem</plugin>
             </hardware>
-            <!-- 左前轮 -->
+            <!-- 左前轮 - 恢复完整控制接口 -->
             <joint name="lfj">
                 <command_interface name="velocity">
@@ -34,5 +34,5 @@
                 <state_interface name="effort" />
             </joint>
-            <!-- 右前轮 -->
+            <!-- 右前轮 - 恢复完整控制接口 -->
             <joint name="rfj">
                 <command_interface name="velocity">
@@ -74,5 +74,5 @@
             </plugin>
         </gazebo>
-        <!-- 为每个轮子关节添加Gazebo插件 -->
+        <!-- 为所有轮子关节添加Gazebo插件 -->
         <gazebo reference="lfj">
             <provideFeedback>true</provideFeedback>
